File: FlexLogic_EVB.kicad_pcb (KiCad board)
At the start: 6 copper layers, 100 x 100 mm, 312 parts, among them IC1 MT9700, IC2 SL2.1s, IC4 LCMXO2-1200HC-4SG32I, IC5 MTS4P, IC6 XT25F32FDTIGT, J1 GT-USB-7010ASV, J11 Conn_02x03_Odd_Even, J12 1.0-3PWB, J13 HB9500M-9.5-4P, J14 TF-CARD_H1.8_SY, J15 HC-FPC-0.5-12P-CXH20, J2 WJ126V-5.0-2P, J3 WJ126V-5.0-2P, J4 WJ126V-5.0-2P, J5 WJ126V-5.0-2P, J6 Conn_02x03_Odd_Even, J7 Conn_02x03_Odd_Even, J8 Conn_02x03_Odd_Even, J9 Conn_02x03_Odd_Even, Q1 L2N7002SLLT1G, Q2 L2N7002SLLT1G, Q4 L2N7002SLLT1G, SW1 QS-301-AGS5P, SW3 DS-04R, U1 RT5752AHGJ5, U10 RQ12000160, U11 RP2350_60QFN, U12 TMUX1574DYYR, U13 ESP-12F, U14 MCP4725xxx-xCH, U15 CC6920SO-10A, U16 CC6920SO-10A, U17 TMUX1574DYYR, U19 LMV321ATDTR, U2 TLV803SDBZR, U20 LMV321ATDTR, U21 ADS1115IDGSR, U22 LMV321ATDTR, U23 LMV321ATDTR, U3 RQ12000160, U4 ADS1115IDGSR, U5 TMUX1574DYYR, U6 RQ12000160, U7 ADS1115IDGSR, U8 FT2232HL, U9 93LC56BT-I

Commit message: 1S commit
Parts:
- removed ? (x2): , 
- removed GND (x2): RH-5001, TestPoint:TestPoint_THTPad_D2.5mm_Drill1.2mm
- removed OUT (x2): RH-5117, TestPoint:TestPoint_THTPad_D2.5mm_Drill1.2mm
- added R13: 4.7k, Resistor_SMD:R_0201_0603Metric_Pad0.64x0.40mm_HandSolder, B.Cu at (114.3, 132.0)
- added TP1: RH-5117, TestPoint:TestPoint_THTPad_D2.5mm_Drill1.2mm, F.Cu at (178.3, 138.7)
- added TP2: RH-5001, TestPoint:TestPoint_THTPad_D2.5mm_Drill1.2mm, F.Cu at (178.3, 133.6)
- added TP4: RH-5117, TestPoint:TestPoint_THTPad_D2.5mm_Drill1.2mm, F.Cu at (178.3, 119.8)
- added TP5: RH-5001, TestPoint:TestPoint_THTPad_D2.5mm_Drill1.2mm, F.Cu at (178.3, 114.7)
- moved S1 3.99 mm to (116.6, 114.8)
- moved R9 2.70 mm to (118.6, 112.5), turned to 0 degrees
- moved J15 2.24 mm to (173.0, 87.7)
- moved C131 2.14 mm to (176.4, 89.2)
- moved C132 2.14 mm to (176.4, 88.5)
- moved C120 2.12 mm to (204.1, 76.6)
- moved R102 2.12 mm to (203.4, 79.1)
- moved R103 2.12 mm to (203.8, 77.8)
- moved R25 0.49 mm to (137.8, 114.2), turned to 90 degrees
Connections:
- U17 pad 10: Net-(U17-D3B) -> unconnected-(U17-D3B-Pad10)
- U17 pad 11: unconnected-(U17-D3A-Pad11) -> Net-(U17-D3A)
- U17 pad 13: Net-(U17-S4B) -> unconnected-(U17-S4B-Pad13)
- U17 pad 14: unconnected-(U17-S4A-Pad14) -> Net-(U17-S4A)
- U17 pad 2: MCU_TXD0 -> Net-(U17-S1A)
- U17 pad 3: Net-(U17-S1B) -> MCU_TXD0
- U17 pad 5: MCU_RXD0 -> Net-(U17-S2A)
- U17 pad 6: Net-(U17-S2B) -> MCU_RXD0
- U5 pad 10: Net-(U17-D3B) -> RTS_N_PIN
- U5 pad 11: RTS_N_PIN -> Net-(U17-D3A)
- U5 pad 13: Net-(U17-S4B) -> CTS_N_PIN
- U5 pad 14: CTS_N_PIN -> Net-(U17-S4A)
- U5 pad 2: TXD_PIN -> Net-(U17-S1A)
- U5 pad 3: Net-(U17-S1B) -> TXD_PIN
- U5 pad 5: RXD_PIN -> Net-(U17-S2A)
- U5 pad 6: Net-(U17-S2B) -> RXD_PIN
Routing:
- net Net-(U17-S1B): track 52.8 -> 0.00 mm, vias 4 -> 0
- net Net-(U17-S1A): track 0.00 -> 52.1 mm, vias 0 -> 4
- net GND: track 184.0 -> 234.3 mm, vias 1077 -> 1087
- net Net-(U17-S2A): track 0.00 -> 40.6 mm, vias 0 -> 4
- net Net-(U17-S4B): track 36.7 -> 0.00 mm, vias 3 -> 0
- net Net-(U17-S2B): track 36.6 -> 0.00 mm, vias 4 -> 0
- net Net-(U17-S4A): track 0.00 -> 34.6 mm, vias 0 -> 2
- net Net-(U17-D3A): track 0.00 -> 33.9 mm
- net Net-(U17-D3B): track 32.9 -> 0.00 mm
- net +3.3V_D: track 118.4 -> 128.2 mm, vias 38 -> 39
- net RTS_N_WIFI: track 59.3 -> 54.3 mm
- net CTS_N_WIFI: track 53.4 -> 56.5 mm
- net TDO_PIN: track 59.4 -> 56.4 mm
- net RESET_N: track 228.9 -> 226.6 mm
- net Net-(R102-Pad1): track 2.38 -> 4.62 mm
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Other:
- board text added: "10A MAX 200mV/A"
- board text removed: "10A MAX"
