File: FlexLogic_EVB.kicad_sch (KiCad schematic)
At the start: 303 parts, among them IC1 MT9700, IC2 SL2.1s, IC4 LCMXO2-1200HC-4SG32I, IC5 MTS4P, IC6 XT25F32FDTIGT, J1 GT-USB-7010ASV, J11 Conn_02x03_Odd_Even, J12 1.0-3PWB, J13 HB9500M-9.5-4P, J14 TF-CARD_H1.8_SY, J15 HC-FPC-0.5-12P-CXH20, J2 WJ126V-5.0-2P, J3 WJ126V-5.0-2P, J4 WJ126V-5.0-2P, J5 WJ126V-5.0-2P, J6 Conn_02x03_Odd_Even, J7 Conn_02x03_Odd_Even, J8 Conn_02x03_Odd_Even, J9 Conn_02x03_Odd_Even, Q1 L2N7002SLLT1G, Q2 L2N7002SLLT1G, Q4 L2N7002SLLT1G, SW1 QS-301-AGS5P, SW3 DS-04R, U1 RT5752AHGJ5, U10 RQ12000160, U11 RP2350_60QFN, U13 ESP-12F, U14 MCP4725xxx-xCH, U15 CC6920SO-10A, U16 CC6920SO-10A, U19 LMV321ATDTR, U2 TLV803SDBZR, U20 LMV321ATDTR, U21 ADS1115IDGSR, U22 LMV321ATDTR, U23 LMV321ATDTR, U3 RQ12000160, U4 ADS1115IDGSR, U6 RQ12000160, U7 ADS1115IDGSR, U8 FT2232HL, U9 93LC56BT-I

Commit message: 1S commit
Parts:
- added R13: 4.7k, Resistor_SMD:R_0201_0603Metric_Pad0.64x0.40mm_HandSolder, symbol Device:R
Connections:
- net +3.3V_FT2232H: now also R13.1
- net UART_SEL: now also R13.2
Other:
- note added: "min:3.24V typ:3.33V max:3.42V 1.454Amax"
- note removed: "min:3.24V typ:3.33V max:3.42V 0.647Amax"
- moved on the sheet: C112, R91
