File: UART Select.kicad_sch (KiCad schematic)
At the start: 4 parts, among them U17 TMUX1574DYYR, U5 TMUX1574DYYR

Commit message: 1S commit
Connections:
- net CTS_N_PIN: now also U5.13 (S4B); no longer U5.14 (S4A)
- net MCU_RXD0: now also U17.6 (S2B); no longer U17.5 (S2A)
- net MCU_TXD0: now also U17.3 (S1B); no longer U17.2 (S1A)
- net RTS_N_PIN: now also U5.10 (D3B); no longer U5.11 (D3A)
- net RXD_PIN: now also U5.6 (S2B); no longer U5.5 (S2A)
- net TXD_PIN: now also U5.3 (S1B); no longer U5.2 (S1A)
- net at U17.10 (D3B): no longer U5.10 (D3B)
- net at U17.11 (D3A): now also U5.11 (D3A)
- net at U17.13 (S4B): no longer U5.13 (S4B)
- net at U17.14 (S4A): now also U5.14 (S4A)
- new net: U17.2 (S1A), U5.2 (S1A)
- new net: U17.5 (S2A), U5.5 (S2A)
